File: Conector grove 4 pinos universal/LDR2/LDR2.kicad_pcb (KiCad board)
At the start: 2 copper layers, 27 x 22.5 mm, 6 parts, among them P4 CON3

Commit message: Connector patch
Parts:
- P4: footprint MY_kicad:molex_2510 -> MyFootprint:Grove 4 pinos
- moved P4 3.61 mm to (28.0, 33.8)
Changed lines of the file:
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@@
   (general
     (links 8)
-    (no_connects 1)
+    (no_connects 0)
     (area 14.924999 14.924999 42.075001 37.575001)
     (thickness 1.6)
     (drawings 12)
-    (tracks 21)
+    (tracks 22)
     (zones 0)
     (modules 6)
@@
   )
   (setup
-    (last_trace_width 0.25)
+    (last_trace_width 1.5)
     (user_trace_width 0.8)
     (user_trace_width 1)
@@
     )
   )
-  (module MY_kicad:molex_2510 (layer F.Cu)
-    (at 24.4 34)
-    (fp_text reference P4 (at 0 -3.81) (layer F.SilkS) hide
-      (effects (font (size 1 1) (thickness 0.15)))
-    )
-    (fp_text value CON3 (at 3.69 -2.43) (layer F.Fab) hide
-      (effects (font (size 1 1) (thickness 0.15)))
-    )
-    (fp_line (start -1.27 1.5) (end 8.89 1.5) (layer F.SilkS) (width 0.15))
-    (fp_line (start -1.27 1.9) (end 8.89 1.9) (layer F.SilkS) (width 0.15))
-    (fp_line (start 8.89 2.5) (end 8.89 -3.2) (layer F.SilkS) (width 0.15))
-    (fp_line (start -1.27 -3.2) (end 8.89 -3.2) (layer F.SilkS) (width 0.15))
-    (fp_line (start -1.27 2.5) (end -1.27 -3.2) (layer F.SilkS) (width 0.15))
-    (fp_line (start -1.27 2.5) (end 8.89 2.5) (layer F.SilkS) (width 0.15))
-    (pad 1 thru_hole oval (at 0 0) (size 2 4) (drill 0.8) (layers *.Cu)
-      (net 3 P6))
-    (pad 2 thru_hole oval (at 2.54 0) (size 2 4) (drill 0.8) (layers *.Cu)
-      (net 2 P5))
-    (pad 3 thru_hole oval (at 5.08 0) (size 2 4) (drill 0.8) (layers *.Cu)
-      (net 7 VCC))
-    (pad 4 thru_hole oval (at 7.62 0) (size 2 4) (drill 0.8) (layers *.Cu)
-      (net 6 GND))
-  )
   (module Resistors_ThroughHole:Resistor_Horizontal_RM10mm (layer F.Cu)
     (at 17 18.5 270)
@@
     )
   )
+  (module "MyFootprint:Grove 4 pinos" (layer F.Cu)
+    (at 28 33.8)
+    (fp_text reference P4 (at -4 -3) (layer F.SilkS) hide
+      (effects (font (size 1 1) (thickness 0.15)))
+    )
+    (fp_text value CON3 (at 0 4) (layer F.Fab) hide
+      (effects (font (size 1 1) (thickness 0.15)))
+    )
+    (fp_line (start -5 2.3) (end 5 2.3) (layer F.SilkS) (width 0.15))
+    (fp_line (start 1.75 2.3) (end 3.39 2.3) (layer F.SilkS) (width 0.15))
+    (fp_line (start 5.01 3) (end 3.39 3) (layer F.SilkS) (width 0.15))
+    (fp_line (start 3.39 3) (end 3.39 2.3) (layer F.SilkS) (width 0.15))
+    (fp_line (start 5 2.3) (end 5 3) (layer F.SilkS) (width 0.15))
+    (fp_line (start -3.38 2.3) (end -1.75 2.3) (layer F.SilkS) (width 0.15))
+    (fp_line (start -4.98 3) (end -3.38 3) (layer F.SilkS) (width 0.15))
+    (fp_line (start -3.38 3) (end -3.38 2.3) (layer F.SilkS) (width 0.15))
+    (fp_line (start -5 2.3) (end -5 3) (layer F.SilkS) (width 0.15))
+    (fp_line (start 1.75 3) (end -1.75 3) (layer F.SilkS) (width 0.15))
+    (fp_line (start 5 2.3) (end 5 -2) (layer F.SilkS) (width 0.15))
+    (fp_line (start -5 -2) (end -5 2.3) (layer F.SilkS) (width 0.15))
+    (fp_line (start 1.75 2.3) (end 1.75 3) (layer F.SilkS) (width 0.15))
+    (fp_line (start -1.75 2.3) (end -1.75 3) (layer F.SilkS) (width 0.15))
+    (fp_line (start -5 -2) (end 5 -2) (layer F.SilkS) (width 0.15))
+    (pad 1 thru_hole oval (at -3 0) (size 1.5 3) (drill 0.8) (layers *.Cu)
+      (net 3 P6))
+    (pad 2 thru_hole oval (at -1 0) (size 1.5 3) (drill 0.8) (layers *.Cu)
+      (net 2 P5))
+    (pad 3 thru_hole oval (at 1 0) (size 1.5 3) (drill 0.8) (layers *.Cu)
+      (net 7 VCC))
+    (pad 4 thru_hole oval (at 3 0) (size 1.5 3) (drill 0.8) (layers *.Cu)
+      (net 6 GND))
+  )
   (gr_text GERSE (at 39.25 16 180) (layer B.Cu)
     (effects (font (size 1 1) (thickness 0.25)) (justify mirror))
@@
   (segment (start 20.28 20.28) (end 23.225 20.28) (width 1.5) (layer B.Cu) (net 1))
   (segment (start 18.5 18.5) (end 20.28 20.28) (width 1.5) (layer B.Cu) (net 1))
+  (segment (start 27 33.8) (end 27 26) (width 1.5) (layer B.Cu) (net 2) (status 400000))
+  (segment (start 28.94 24.06) (end 28.94 20.28) (width 1.5) (layer B.Cu) (net 2) (status 800000))
+  (segment (start 27 26) (end 28.94 24.06) (width 1.5) (layer B.Cu) (net 2))
   (segment (start 40 24) (end 40 21) (width 1.5) (layer B.Cu) (net 2))
   (segment (start 28.94 18.56) (end 28.94 20.28) (width 1.5) (layer B.Cu) (net 2))
@@
   (segment (start 36.5 17.5) (end 30 17.5) (width 1.5) (layer B.Cu) (net 2))
   (segment (start 40 21) (end 36.5 17.5) (width 1.5) (layer B.Cu) (net 2))
-  (segment (start 28.94 24.06) (end 28.94 20.28) (width 1.5) (layer B.Cu) (net 2))
   (segment (start 28.94 20.28) (end 28.94 19.56) (width 0.8) (layer B.Cu) (net 2))
-  (segment (start 26.92 26.08) (end 28.94 24.06) (width 1.5) (layer B.Cu) (net 2))
-  (segment (start 26.92 33.5) (end 26.92 26.08) (width 1.5) (layer B.Cu) (net 2))
-  (segment (start 25.765 22.735) (end 25.765 20.28) (width 1.5) (layer B.Cu) (net 3))
-  (segment (start 24.38 24.12) (end 25.765 22.735) (width 1.5) (layer B.Cu) (net 3))
-  (segment (start 24.38 33.5) (end 24.38 24.12) (width 1.5) (layer B.Cu) (net 3))
+  (segment (start 25.765 20.28) (end 25.765 23.435) (width 1.5) (layer B.Cu) (net 3) (status 400000))
+  (segment (start 25 24.2) (end 25 33.8) (width 1.5) (layer B.Cu) (net 3) (status 800000))
+  (segment (start 25.765 23.435) (end 25 24.2) (width 1.5) (layer B.Cu) (net 3))
   (segment (start 32 29) (end 37.46128 29) (width 2) (layer B.Cu) (net 4))
   (segment (start 37.46128 29) (end 37.50064 29.03936) (width 2) (layer B.Cu) (net 4))
-  (segment (start 29.46 33.5) (end 29.46 27.54) (width 1.5) (layer B.Cu) (net 7))
-  (segment (start 29.46 27.54) (end 31 26) (width 1.5) (layer B.Cu) (net 7))
-  (segment (start 31 26) (end 31 22.03) (width 1.5) (layer B.Cu) (net 7))
-  (segment (start 31 22.03) (end 32.75 20.28) (width 1.5) (layer B.Cu) (net 7))
+  (segment (start 32.75 20.28) (end 32.75 20.65) (width 1.5) (layer B.Cu) (net 7) (status C00000))
+  (segment (start 32.75 20.65) (end 31.2 22.2) (width 1.5) (layer B.Cu) (net 7) (status 400000))
+  (segment (start 31.2 22.2) (end 31.2 25.6) (width 1.5) (layer B.Cu) (net 7))
+  (segment (start 31.2 25.6) (end 29 27.8) (width 1.5) (layer B.Cu) (net 7))
+  (segment (start 29 27.8) (end 29 33.8) (width 1.5) (layer B.Cu) (net 7) (status 800000))
   (zone (net 6) (net_name GND) (layer B.Cu) (hatch edge 0.508)
     (connect_pads yes (clearance 0.5))
