File: Conector grove 4 pinos universal/LDR2/LDR2.sch (KiCad schematic (older format))
At the start: 6 parts, among them P4 CON3

Commit message: Connector patch
Parts:
- P4: footprint MY_kicad:molex_2510 -> MyFootprint:Grove 4 pinos
- R7: footprint MY_kicad:LDR3mm -> MyFootprint:LDR3mm
Changed lines of the file:
@@
 F 0 "P4" H 4950 1050 50  0000 C CNN
 F 1 "CON3" V 5050 1300 50  0000 C CNN
-F 2 "MY_kicad:molex_2510" H 4950 1300 50  0001 C CNN
+F 2 "MyFootprint:Grove 4 pinos" H 4950 1300 50  0001 C CNN
 F 3 "" H 4950 1300 50  0000 C CNN
 	1    4950 1300
@@
 F 0 "R7" V 5700 2000 50  0000 C CNN
 F 1 "LDR-3MM" V 5900 2000 50  0000 C TNN
-F 2 "MY_kicad:LDR3mm" V 5730 2000 50  0001 C CNN
+F 2 "MyFootprint:LDR3mm" V 5730 2000 50  0001 C CNN
 F 3 "" H 5800 2000 50  0000 C CNN
 	1    5800 2000
