File: Conector molex 2510 4 pinos/Botao/Botao.kicad_pcb (KiCad board)
At the start: 2 copper layers, 265 x 145 mm, 162 parts, among them P6 CON5, SW1 SW_PUSH, SW2 SP6T

Commit message: Connector patch
Parts:
- removed the P6 at (271.0, 155.0)
- removed the P6 at (151.0, 80.0)
- removed the P6 at (151.0, 130.0)
- removed the P6 at (151.0, 155.0)
- removed the P6 at (181.0, 155.0)
- removed the P6 at (181.0, 130.0)
- removed the P6 at (181.0, 80.0)
- removed the P6 at (181.0, 105.0)
- removed the P6 at (181.0, 55.0)
- removed the P6 at (181.0, 30.0)
- removed the P6 at (241.0, 30.0)
- removed the P6 at (271.0, 130.0)
- removed the P6 at (241.0, 55.0)
- removed the P6 at (241.0, 105.0)
- removed the P6 at (241.0, 80.0)
- removed the P6 at (241.0, 130.0)
- removed the P6 at (241.0, 155.0)
- removed the P6 at (211.0, 155.0)
- removed the P6 at (211.0, 130.0)
- removed the P6 at (211.0, 80.0)
- removed the P6 at (211.0, 105.0)
- removed the P6 at (211.0, 55.0)
- removed the P6 at (271.0, 80.0)
- removed the P6 at (211.0, 30.0)
- removed the P6 at (91.0, 30.0)
- removed the P6 at (91.0, 55.0)
- removed the P6 at (91.0, 105.0)
- removed the P6 at (91.0, 80.0)
- removed the P6 at (91.0, 130.0)
- removed the P6 at (91.0, 155.0)
- removed the P6 at (121.0, 155.0)
- removed the P6 at (121.0, 130.0)
- removed the P6 at (121.0, 80.0)
- removed the P6 at (271.0, 105.0)
- removed the P6 at (121.0, 105.0)
- removed the P6 at (121.0, 55.0)
- removed the P6 at (121.0, 30.0)
- removed the P6 at (61.0, 30.0)
- removed the P6 at (61.0, 55.0)
- removed the P6 at (61.0, 105.0)
- removed the P6 at (61.0, 80.0)
- removed the P6 at (61.0, 130.0)
- removed the P6 at (61.0, 155.0)
- removed the P6 at (31.0, 155.0)
- removed the P6 at (271.0, 55.0)
- removed the P6 at (31.0, 130.0)
- removed the P6 at (31.0, 80.0)
- removed the P6 at (31.0, 105.0)
- removed the P6 at (31.0, 55.0)
- removed the P6 at (271.0, 30.0)
- removed the P6 at (151.0, 30.0)
- removed the P6 at (151.0, 55.0)
- removed the P6 at (151.0, 105.0)
- removed the SW1 at (273.7, 146.6)
- removed the SW1 at (153.7, 71.6)
- removed the SW1 at (153.7, 121.6)
- removed the SW1 at (153.7, 146.6)
- removed the SW1 at (183.7, 146.6)
- removed the SW1 at (183.7, 121.6)
- removed the SW1 at (183.7, 71.6)
- removed the SW1 at (183.7, 96.6)
- removed the SW1 at (183.7, 46.6)
- removed the SW1 at (183.7, 21.6)
- removed the SW1 at (243.7, 21.6)
- removed the SW1 at (273.7, 121.6)
- removed the SW1 at (243.7, 46.6)
- removed the SW1 at (243.7, 96.6)
- removed the SW1 at (243.7, 71.6)
- removed the SW1 at (243.7, 121.6)
- removed the SW1 at (243.7, 146.6)
- removed the SW1 at (213.7, 146.6)
- removed the SW1 at (213.7, 121.6)
- removed the SW1 at (213.7, 71.6)
- removed the SW1 at (213.7, 96.6)
- removed the SW1 at (213.7, 46.6)
- removed the SW1 at (273.7, 71.6)
- removed the SW1 at (213.7, 21.6)
- removed the SW1 at (93.7, 21.6)
- removed the SW1 at (93.7, 46.6)
- removed the SW1 at (93.7, 96.6)
- removed the SW1 at (93.7, 71.6)
- removed the SW1 at (93.7, 121.6)
- removed the SW1 at (93.7, 146.6)
- removed the SW1 at (123.7, 146.6)
- removed the SW1 at (123.7, 121.6)
- removed the SW1 at (123.7, 71.6)
- removed the SW1 at (273.7, 96.6)
- removed the SW1 at (123.7, 96.6)
- removed the SW1 at (123.7, 46.6)
- removed the SW1 at (123.7, 21.6)
- removed the SW1 at (63.7, 21.6)
- removed the SW1 at (63.7, 46.6)
- removed the SW1 at (63.7, 96.6)
- removed the SW1 at (63.7, 71.6)
- removed the SW1 at (63.7, 121.6)
- removed the SW1 at (63.7, 146.6)
- removed the SW1 at (33.7, 146.6)
- removed the SW1 at (273.7, 46.6)
- removed the SW1 at (33.7, 121.6)
- removed the SW1 at (33.7, 71.6)
- removed the SW1 at (33.7, 96.6)
- removed the SW1 at (33.7, 46.6)
- removed the SW1 at (273.7, 21.6)
- removed the SW1 at (153.7, 21.6)
- removed the SW1 at (153.7, 46.6)
- removed the SW1 at (153.7, 96.6)
- removed the SW2 at (258.5, 144.0)
- removed the SW2 at (138.5, 69.0)
- removed the SW2 at (138.5, 119.0)
- removed the SW2 at (138.5, 144.0)
- removed the SW2 at (168.5, 144.0)
- removed the SW2 at (168.5, 119.0)
- removed the SW2 at (168.5, 69.0)
- removed the SW2 at (168.5, 94.0)
- removed the SW2 at (168.5, 44.0)
- removed the SW2 at (168.5, 19.0)
- removed the SW2 at (228.5, 19.0)
- removed the SW2 at (258.5, 119.0)
- removed the SW2 at (228.5, 44.0)
- removed the SW2 at (228.5, 94.0)
- removed the SW2 at (228.5, 69.0)
- removed the SW2 at (228.5, 119.0)
- removed the SW2 at (228.5, 144.0)
- removed the SW2 at (198.5, 144.0)
- removed the SW2 at (198.5, 119.0)
- removed the SW2 at (198.5, 69.0)
- removed the SW2 at (198.5, 94.0)
- removed the SW2 at (198.5, 44.0)
- removed the SW2 at (258.5, 69.0)
- removed the SW2 at (198.5, 19.0)
- removed the SW2 at (78.5, 19.0)
- removed the SW2 at (78.5, 44.0)
- removed the SW2 at (78.5, 94.0)
- removed the SW2 at (78.5, 69.0)
- removed the SW2 at (78.5, 119.0)
- removed the SW2 at (78.5, 144.0)
- removed the SW2 at (108.5, 144.0)
- removed the SW2 at (108.5, 119.0)
- removed the SW2 at (108.5, 69.0)
- removed the SW2 at (258.5, 94.0)
- removed the SW2 at (108.5, 94.0)
- removed the SW2 at (108.5, 44.0)
- removed the SW2 at (108.5, 19.0)
- removed the SW2 at (48.5, 19.0)
- removed the SW2 at (48.5, 44.0)
- removed the SW2 at (48.5, 94.0)
- removed the SW2 at (48.5, 69.0)
- removed the SW2 at (48.5, 119.0)
- removed the SW2 at (48.5, 144.0)
- removed the SW2 at (18.5, 144.0)
- removed the SW2 at (258.5, 44.0)
- removed the SW2 at (18.5, 119.0)
- removed the SW2 at (18.5, 69.0)
- removed the SW2 at (18.5, 94.0)
- removed the SW2 at (18.5, 44.0)
- removed the SW2 at (258.5, 19.0)
- removed the SW2 at (138.5, 19.0)
- removed the SW2 at (138.5, 44.0)
- removed the SW2 at (138.5, 94.0)
- moved P6 7.57 mm to (23.4, 29.8), turned to 0 degrees
Connections:
- P6 pad 1: P9 -> GND
- P6 pad 2: P10 -> VCC
- P6 pad 3: VCC -> P10
- P6 pad 4: GND -> P9
Routing:
- net P10: track 1148.0 -> 21.3 mm
- net VCC: track 679.8 -> 12.6 mm
- net P9: track 520.4 -> 9.64 mm
Other:
- board size 265 x 145 mm -> 25 x 20 mm
- board text removed: "Não é necessario espelhar, imagem F.Silks já espelhada... No need to mirror, F.Silks image already mirrored ..."
