File: Conector molex 2510 4 pinos/Botao/Botao.sch (KiCad schematic (older format))
At the start: 3 parts, among them P6 CON5, SW1 SW_PUSH, SW2 SP6T

Commit message: Connector patch
Connections:
- net GND: now also P6.1 (P1); no longer P6.4 (P4)
- net P10: now also P6.3 (P3); no longer P6.2 (P2)
- net P9: now also P6.4 (P4); no longer P6.1 (P1)
- net VCC: now also P6.2 (P2); no longer P6.3 (P3)
