File: Conector molex 2510 4 pinos/BotaoADC/BotaoADC.kicad_pcb (KiCad board)
At the start: 2 copper layers, 245 x 155 mm, 280 parts, among them P7 CON6, SW3 SW_PUSH, SW4 SW_PUSH, SW5 SW_PUSH, SW6 SW_PUSH, SW7 SW_PUSH, SW8 SW_PUSH

Commit message: Connector patch
Parts:
- removed the G*** at (248.5, 121.0)
- removed the G*** at (198.5, 81.0)
- removed the G*** at (198.5, 161.0)
- removed the G*** at (198.5, 121.0)
- removed the G*** at (98.5, 121.0)
- removed the G*** at (98.5, 161.0)
- removed the G*** at (98.5, 81.0)
- removed the G*** at (98.5, 41.0)
- removed the G*** at (48.5, 81.0)
- removed the G*** at (48.5, 161.0)
- removed the G*** at (248.5, 161.0)
- removed the G*** at (48.5, 121.0)
- removed the G*** at (248.5, 81.0)
- removed the G*** at (248.5, 41.0)
- removed the G*** at (148.5, 121.0)
- removed the G*** at (148.5, 161.0)
- removed the G*** at (148.5, 81.0)
- removed the G*** at (148.5, 41.0)
- removed the G*** at (198.5, 41.0)
- removed the P7 at (233.0, 126.0)
- removed the P7 at (183.0, 86.0)
- removed the P7 at (183.0, 166.0)
- removed the P7 at (183.0, 126.0)
- removed the P7 at (83.0, 126.0)
- removed the P7 at (83.0, 166.0)
- removed the P7 at (83.0, 86.0)
- removed the P7 at (83.0, 46.0)
- removed the P7 at (33.0, 86.0)
- removed the P7 at (33.0, 166.0)
- removed the P7 at (233.0, 166.0)
- removed the P7 at (33.0, 126.0)
- removed the P7 at (233.0, 86.0)
- removed the P7 at (233.0, 46.0)
- removed the P7 at (133.0, 126.0)
- removed the P7 at (133.0, 166.0)
- removed the P7 at (133.0, 86.0)
- removed the P7 at (133.0, 46.0)
- removed the P7 at (183.0, 46.0)
- removed the R10 at (231.1, 105.2)
- removed the R10 at (181.1, 65.2)
- removed the R10 at (181.1, 145.2)
- removed the R10 at (181.1, 105.2)
- removed the R10 at (81.1, 105.2)
- removed the R10 at (81.1, 145.2)
- removed the R10 at (81.1, 65.2)
- removed the R10 at (81.1, 25.2)
- removed the R10 at (31.1, 65.2)
- removed the R10 at (31.1, 145.2)
- removed the R10 at (231.1, 145.2)
- removed the R10 at (31.1, 105.2)
- removed the R10 at (231.1, 65.2)
- removed the R10 at (231.1, 25.2)
- removed the R10 at (131.1, 105.2)
- removed the R10 at (131.1, 145.2)
- removed the R10 at (131.1, 65.2)
- removed the R10 at (131.1, 25.2)
- removed the R10 at (181.1, 25.2)
- removed the R11 at (231.1, 102.1)
- removed the R11 at (181.1, 62.1)
- removed the R11 at (181.1, 142.1)
- removed the R11 at (181.1, 102.1)
- removed the R11 at (81.1, 102.1)
- removed the R11 at (81.1, 142.1)
- removed the R11 at (81.1, 62.1)
- removed the R11 at (81.1, 22.1)
- removed the R11 at (31.1, 62.1)
- removed the R11 at (31.1, 142.1)
- removed the R11 at (231.1, 142.1)
- removed the R11 at (31.1, 102.1)
- removed the R11 at (231.1, 62.1)
- removed the R11 at (231.1, 22.1)
- removed the R11 at (131.1, 102.1)
- removed the R11 at (131.1, 142.1)
- removed the R11 at (131.1, 62.1)
- removed the R11 at (131.1, 22.1)
- removed the R11 at (181.1, 22.1)
- removed the R12 at (244.5, 102.1)
- removed the R12 at (194.5, 62.1)
- removed the R12 at (194.5, 142.1)
- removed the R12 at (194.5, 102.1)
- removed the R12 at (94.5, 102.1)
- removed the R12 at (94.5, 142.1)
- removed the R12 at (94.5, 62.1)
- removed the R12 at (94.5, 22.1)
- removed the R12 at (44.5, 62.1)
- removed the R12 at (44.5, 142.1)
- removed the R12 at (244.5, 142.1)
- removed the R12 at (44.5, 102.1)
- removed the R12 at (244.5, 62.1)
- removed the R12 at (244.5, 22.1)
- removed the R12 at (144.5, 102.1)
- removed the R12 at (144.5, 142.1)
- removed the R12 at (144.5, 62.1)
- removed the R12 at (144.5, 22.1)
- removed the R12 at (194.5, 22.1)
- removed the R13 at (254.6, 105.2)
- removed the R13 at (204.6, 65.2)
- removed the R13 at (204.6, 145.2)
- removed the R13 at (204.6, 105.2)
- removed the R13 at (104.6, 105.2)
- removed the R13 at (104.6, 145.2)
- removed the R13 at (104.6, 65.2)
- removed the R13 at (104.6, 25.2)
- removed the R13 at (54.6, 65.2)
- removed the R13 at (54.6, 145.2)
- removed the R13 at (254.6, 145.2)
- removed the R13 at (54.6, 105.2)
- removed the R13 at (254.6, 65.2)
- removed the R13 at (254.6, 25.2)
- removed the R13 at (154.6, 105.2)
- removed the R13 at (154.6, 145.2)
- removed the R13 at (154.6, 65.2)
- removed the R13 at (154.6, 25.2)
- removed the R13 at (204.6, 25.2)
- removed the R8 at (217.3, 105.2)
- removed the R8 at (167.3, 65.2)
- removed the R8 at (167.3, 145.2)
- removed the R8 at (167.3, 105.2)
- removed the R8 at (67.3, 105.2)
- removed the R8 at (67.3, 145.2)
- removed the R8 at (67.3, 65.2)
- removed the R8 at (67.3, 25.2)
- removed the R8 at (17.3, 65.2)
- removed the R8 at (17.3, 145.2)
- removed the R8 at (217.3, 145.2)
- removed the R8 at (17.3, 105.2)
- removed the R8 at (217.3, 65.2)
- removed the R8 at (217.3, 25.2)
- removed the R8 at (117.3, 105.2)
- removed the R8 at (117.3, 145.2)
- removed the R8 at (117.3, 65.2)
- removed the R8 at (117.3, 25.2)
- removed the R8 at (167.3, 25.2)
- removed the R9 at (217.3, 102.1)
- removed the R9 at (167.3, 62.1)
- removed the R9 at (167.3, 142.1)
- removed the R9 at (167.3, 102.1)
- removed the R9 at (67.3, 102.1)
- removed the R9 at (67.3, 142.1)
- removed the R9 at (67.3, 62.1)
- removed the R9 at (67.3, 22.1)
- removed the R9 at (17.3, 62.1)
- removed the R9 at (17.3, 142.1)
- removed the R9 at (217.3, 142.1)
- removed the R9 at (17.3, 102.1)
- removed the R9 at (217.3, 62.1)
- removed the R9 at (217.3, 22.1)
- removed the R9 at (117.3, 102.1)
- removed the R9 at (117.3, 142.1)
- removed the R9 at (117.3, 62.1)
- removed the R9 at (117.3, 22.1)
- removed the R9 at (167.3, 22.1)
- removed the SW3 at (219.0, 113.0)
- removed the SW3 at (169.0, 73.0)
- removed the SW3 at (169.0, 153.0)
- removed the SW3 at (169.0, 113.0)
- removed the SW3 at (69.0, 113.0)
- removed the SW3 at (69.0, 153.0)
- removed the SW3 at (69.0, 73.0)
- removed the SW3 at (69.0, 33.0)
- removed the SW3 at (19.0, 73.0)
- removed the SW3 at (19.0, 153.0)
- removed the SW3 at (219.0, 153.0)
- removed the SW3 at (19.0, 113.0)
- removed the SW3 at (219.0, 73.0)
- removed the SW3 at (219.0, 33.0)
- removed the SW3 at (119.0, 113.0)
- removed the SW3 at (119.0, 153.0)
- removed the SW3 at (119.0, 73.0)
- removed the SW3 at (119.0, 33.0)
- removed the SW3 at (169.0, 33.0)
- removed the SW4 at (226.0, 113.0)
- removed the SW4 at (176.0, 73.0)
- removed the SW4 at (176.0, 153.0)
- removed the SW4 at (176.0, 113.0)
- removed the SW4 at (76.0, 113.0)
- removed the SW4 at (76.0, 153.0)
- removed the SW4 at (76.0, 73.0)
- removed the SW4 at (76.0, 33.0)
- removed the SW4 at (26.0, 73.0)
- removed the SW4 at (26.0, 153.0)
- removed the SW4 at (226.0, 153.0)
- removed the SW4 at (26.0, 113.0)
- removed the SW4 at (226.0, 73.0)
- removed the SW4 at (226.0, 33.0)
- removed the SW4 at (126.0, 113.0)
- removed the SW4 at (126.0, 153.0)
- removed the SW4 at (126.0, 73.0)
- removed the SW4 at (126.0, 33.0)
- removed the SW4 at (176.0, 33.0)
- removed the SW5 at (233.0, 113.0)
- removed the SW5 at (183.0, 73.0)
- removed the SW5 at (183.0, 153.0)
- removed the SW5 at (183.0, 113.0)
- removed the SW5 at (83.0, 113.0)
- removed the SW5 at (83.0, 153.0)
- removed the SW5 at (83.0, 73.0)
- removed the SW5 at (83.0, 33.0)
- removed the SW5 at (33.0, 73.0)
- removed the SW5 at (33.0, 153.0)
- removed the SW5 at (233.0, 153.0)
- removed the SW5 at (33.0, 113.0)
- removed the SW5 at (233.0, 73.0)
- removed the SW5 at (233.0, 33.0)
- removed the SW5 at (133.0, 113.0)
- removed the SW5 at (133.0, 153.0)
- removed the SW5 at (133.0, 73.0)
- removed the SW5 at (133.0, 33.0)
- removed the SW5 at (183.0, 33.0)
- removed the SW6 at (240.0, 113.0)
- removed the SW6 at (190.0, 73.0)
- removed the SW6 at (190.0, 153.0)
- removed the SW6 at (190.0, 113.0)
- removed the SW6 at (90.0, 113.0)
- removed the SW6 at (90.0, 153.0)
- removed the SW6 at (90.0, 73.0)
- removed the SW6 at (90.0, 33.0)
- removed the SW6 at (40.0, 73.0)
- removed the SW6 at (40.0, 153.0)
- removed the SW6 at (240.0, 153.0)
- removed the SW6 at (40.0, 113.0)
- removed the SW6 at (240.0, 73.0)
- removed the SW6 at (240.0, 33.0)
- removed the SW6 at (140.0, 113.0)
- removed the SW6 at (140.0, 153.0)
- removed the SW6 at (140.0, 73.0)
- removed the SW6 at (140.0, 33.0)
- removed the SW6 at (190.0, 33.0)
- removed the SW7 at (247.0, 113.0)
- removed the SW7 at (197.0, 73.0)
- removed the SW7 at (197.0, 153.0)
- removed the SW7 at (197.0, 113.0)
- removed the SW7 at (97.0, 113.0)
- removed the SW7 at (97.0, 153.0)
- removed the SW7 at (97.0, 73.0)
- removed the SW7 at (97.0, 33.0)
- removed the SW7 at (47.0, 73.0)
- removed the SW7 at (47.0, 153.0)
- removed the SW7 at (247.0, 153.0)
- removed the SW7 at (47.0, 113.0)
- removed the SW7 at (247.0, 73.0)
- removed the SW7 at (247.0, 33.0)
- removed the SW7 at (147.0, 113.0)
- removed the SW7 at (147.0, 153.0)
- removed the SW7 at (147.0, 73.0)
- removed the SW7 at (147.0, 33.0)
- removed the SW7 at (197.0, 33.0)
- removed the SW8 at (254.0, 113.0)
- removed the SW8 at (204.0, 73.0)
- removed the SW8 at (204.0, 153.0)
- removed the SW8 at (204.0, 113.0)
- removed the SW8 at (104.0, 113.0)
- removed the SW8 at (104.0, 153.0)
- removed the SW8 at (104.0, 73.0)
- removed the SW8 at (104.0, 33.0)
- removed the SW8 at (54.0, 73.0)
- removed the SW8 at (54.0, 153.0)
- removed the SW8 at (254.0, 153.0)
- removed the SW8 at (54.0, 113.0)
- removed the SW8 at (254.0, 73.0)
- removed the SW8 at (254.0, 33.0)
- removed the SW8 at (154.0, 113.0)
- removed the SW8 at (154.0, 153.0)
- removed the SW8 at (154.0, 73.0)
- removed the SW8 at (154.0, 33.0)
- removed the SW8 at (204.0, 33.0)
- added G***: LOGO, MyFootprint:Logo-IFSP, F.Cu at (26.0, 41.8)
Routing:
- net P11: track 1126.4 -> 56.3 mm
- net BT1: track 921.2 -> 46.1 mm
- net BT2: track 368.9 -> 18.4 mm
- net BT4: track 354.7 -> 17.7 mm
- net BT5: track 240.2 -> 12.0 mm
- net BT3: track 204.1 -> 10.2 mm
- net BT6: track 147.3 -> 7.36 mm
Other:
- board size 245 x 155 mm -> 45 x 35 mm
- board text removed: "Não é necessario espelhar, imagem F.Silks já espelhada... No need to mirror, F.Silks image already mirrored ..."
