File: Conector molex 2510 4 pinos/DHT11/DHT11.kicad_pcb (KiCad board)
At the start: 2 copper layers, 235 x 170 mm, 126 parts, among them P1 DHT11, U1 DHT11

Commit message: Connector patch
Parts:
- removed the P1 at (162.4, 31.8)
- removed the P1 at (197.4, 91.8)
- removed the P1 at (197.4, 61.8)
- removed the P1 at (197.4, 31.8)
- removed the P1 at (232.4, 181.8)
- removed the P1 at (232.4, 151.8)
- removed the P1 at (232.4, 121.8)
- removed the P1 at (232.4, 91.8)
- removed the P1 at (232.4, 61.8)
- removed the P1 at (232.4, 31.8)
- removed the P1 at (92.4, 31.8)
- removed the P1 at (162.4, 61.8)
- removed the P1 at (92.4, 61.8)
- removed the P1 at (92.4, 91.8)
- removed the P1 at (92.4, 121.8)
- removed the P1 at (92.4, 151.8)
- removed the P1 at (92.4, 181.8)
- removed the P1 at (127.4, 181.8)
- removed the P1 at (127.4, 151.8)
- removed the P1 at (127.4, 121.8)
- removed the P1 at (127.4, 91.8)
- removed the P1 at (127.4, 61.8)
- removed the P1 at (162.4, 91.8)
- removed the P1 at (127.4, 31.8)
- removed the P1 at (57.4, 31.8)
- removed the P1 at (57.4, 61.8)
- removed the P1 at (57.4, 91.8)
- removed the P1 at (57.4, 121.8)
- removed the P1 at (57.4, 151.8)
- removed the P1 at (57.4, 181.8)
- removed the P1 at (22.4, 181.8)
- removed the P1 at (22.4, 151.8)
- removed the P1 at (22.4, 121.8)
- removed the P1 at (162.4, 121.8)
- removed the P1 at (22.4, 91.8)
- removed the P1 at (22.4, 61.8)
- removed the P1 at (162.4, 151.8)
- removed the P1 at (162.4, 181.8)
- removed the P1 at (197.4, 181.8)
- removed the P1 at (197.4, 151.8)
- removed the P1 at (197.4, 121.8)
- removed the R1 at (158.0, 18.0)
- removed the R1 at (193.0, 78.0)
- removed the R1 at (193.0, 48.0)
- removed the R1 at (193.0, 18.0)
- removed the R1 at (228.0, 168.0)
- removed the R1 at (228.0, 138.0)
- removed the R1 at (228.0, 108.0)
- removed the R1 at (228.0, 78.0)
- removed the R1 at (228.0, 48.0)
- removed the R1 at (228.0, 18.0)
- removed the R1 at (88.0, 18.0)
- removed the R1 at (158.0, 48.0)
- removed the R1 at (88.0, 48.0)
- removed the R1 at (88.0, 78.0)
- removed the R1 at (88.0, 108.0)
- removed the R1 at (88.0, 138.0)
- removed the R1 at (88.0, 168.0)
- removed the R1 at (123.0, 168.0)
- removed the R1 at (123.0, 138.0)
- removed the R1 at (123.0, 108.0)
- removed the R1 at (123.0, 78.0)
- removed the R1 at (123.0, 48.0)
- removed the R1 at (158.0, 78.0)
- removed the R1 at (123.0, 18.0)
- removed the R1 at (53.0, 18.0)
- removed the R1 at (53.0, 48.0)
- removed the R1 at (53.0, 78.0)
- removed the R1 at (53.0, 108.0)
- removed the R1 at (53.0, 138.0)
- removed the R1 at (53.0, 168.0)
- removed the R1 at (18.0, 168.0)
- removed the R1 at (18.0, 138.0)
- removed the R1 at (18.0, 108.0)
- removed the R1 at (158.0, 108.0)
- removed the R1 at (18.0, 78.0)
- removed the R1 at (18.0, 48.0)
- removed the R1 at (158.0, 138.0)
- removed the R1 at (158.0, 168.0)
- removed the R1 at (193.0, 168.0)
- removed the R1 at (193.0, 138.0)
- removed the R1 at (193.0, 108.0)
- removed the U1 at (165.0, 28.0)
- removed the U1 at (200.0, 88.0)
- removed the U1 at (200.0, 58.0)
- removed the U1 at (200.0, 28.0)
- removed the U1 at (235.0, 178.0)
- removed the U1 at (235.0, 148.0)
- removed the U1 at (235.0, 118.0)
- removed the U1 at (235.0, 88.0)
- removed the U1 at (235.0, 58.0)
- removed the U1 at (235.0, 28.0)
- removed the U1 at (95.0, 28.0)
- removed the U1 at (165.0, 58.0)
- removed the U1 at (95.0, 58.0)
- removed the U1 at (95.0, 88.0)
- removed the U1 at (95.0, 118.0)
- removed the U1 at (95.0, 148.0)
- removed the U1 at (95.0, 178.0)
- removed the U1 at (130.0, 178.0)
- removed the U1 at (130.0, 148.0)
- removed the U1 at (130.0, 118.0)
- removed the U1 at (130.0, 88.0)
- removed the U1 at (130.0, 58.0)
- removed the U1 at (165.0, 88.0)
- removed the U1 at (130.0, 28.0)
- removed the U1 at (60.0, 28.0)
- removed the U1 at (60.0, 58.0)
- removed the U1 at (60.0, 88.0)
- removed the U1 at (60.0, 118.0)
- removed the U1 at (60.0, 148.0)
- removed the U1 at (60.0, 178.0)
- removed the U1 at (25.0, 178.0)
- removed the U1 at (25.0, 148.0)
- removed the U1 at (25.0, 118.0)
- removed the U1 at (165.0, 118.0)
- removed the U1 at (25.0, 88.0)
- removed the U1 at (25.0, 58.0)
- removed the U1 at (165.0, 148.0)
- removed the U1 at (165.0, 178.0)
- removed the U1 at (200.0, 178.0)
- removed the U1 at (200.0, 148.0)
- removed the U1 at (200.0, 118.0)
Routing:
- net VCC: track 1050.5 -> 25.0 mm
- net DHT11: track 822.4 -> 19.6 mm
Other:
- board size 235 x 170 mm -> 25 x 20 mm
- board text removed: "Não é necessario espelhar, imagem F.Silks já espelhada... No need to mirror, F.Silks image already mirrored ..."
