File: Conector molex 2510 4 pinos/HC-SR04/HC-SR04.kicad_pcb (KiCad board)
At the start: 2 copper layers, 204 x 170 mm, 60 parts, among them P2 CON1, U2 HC-SR04

Commit message: Connector patch
Parts:
- removed the P2 at (172.0, 189.0)
- removed the P2 at (127.0, 129.0)
- removed the P2 at (127.0, 99.0)
- removed the P2 at (127.0, 189.0)
- removed the P2 at (127.0, 159.0)
- removed the P2 at (172.0, 159.0)
- removed the P2 at (172.0, 99.0)
- removed the P2 at (172.0, 129.0)
- removed the P2 at (172.0, 69.0)
- removed the P2 at (172.0, 39.0)
- removed the P2 at (82.0, 39.0)
- removed the P2 at (217.0, 189.0)
- removed the P2 at (82.0, 69.0)
- removed the P2 at (82.0, 129.0)
- removed the P2 at (82.0, 99.0)
- removed the P2 at (82.0, 189.0)
- removed the P2 at (82.0, 159.0)
- removed the P2 at (37.0, 159.0)
- removed the P2 at (37.0, 189.0)
- removed the P2 at (37.0, 99.0)
- removed the P2 at (37.0, 129.0)
- removed the P2 at (37.0, 69.0)
- removed the P2 at (217.0, 39.0)
- removed the P2 at (217.0, 69.0)
- removed the P2 at (217.0, 129.0)
- removed the P2 at (217.0, 99.0)
- removed the P2 at (217.0, 159.0)
- removed the P2 at (127.0, 39.0)
- removed the P2 at (127.0, 69.0)
- removed the U2 at (168.0, 178.0)
- removed the U2 at (123.0, 118.0)
- removed the U2 at (123.0, 88.0)
- removed the U2 at (123.0, 178.0)
- removed the U2 at (123.0, 148.0)
- removed the U2 at (168.0, 148.0)
- removed the U2 at (168.0, 88.0)
- removed the U2 at (168.0, 118.0)
- removed the U2 at (168.0, 58.0)
- removed the U2 at (168.0, 28.0)
- removed the U2 at (78.0, 28.0)
- removed the U2 at (213.0, 178.0)
- removed the U2 at (78.0, 58.0)
- removed the U2 at (78.0, 118.0)
- removed the U2 at (78.0, 88.0)
- removed the U2 at (78.0, 178.0)
- removed the U2 at (78.0, 148.0)
- removed the U2 at (33.0, 148.0)
- removed the U2 at (33.0, 178.0)
- removed the U2 at (33.0, 88.0)
- removed the U2 at (33.0, 118.0)
- removed the U2 at (33.0, 58.0)
- removed the U2 at (213.0, 28.0)
- removed the U2 at (213.0, 58.0)
- removed the U2 at (213.0, 118.0)
- removed the U2 at (213.0, 88.0)
- removed the U2 at (213.0, 148.0)
- removed the U2 at (123.0, 28.0)
- removed the U2 at (123.0, 58.0)
- moved P2 7.62 mm to (29.4, 39.6), turned to 0 degrees
Connections:
- P2 pad 1: GND -> P2
- P2 pad 2: VCC -> P1
- P2 pad 3: P1 -> VCC
- P2 pad 4: P2 -> GND
Routing:
- net VCC: track 378.3 -> 12.6 mm
- net P1: track 378.3 -> 12.6 mm
- net P2: track 378.3 -> 12.6 mm
Other:
- board size 204 x 170 mm -> 24 x 20 mm
- board text removed: "Não é necessario espelhar, imagem F.Silks já espelhada... No need to mirror, F.Silks image already mirrored ..."
