File: Conector molex 2510 4 pinos/HC-SR04/HC-SR04.sch (KiCad schematic (older format))
At the start: 2 parts, among them P2 CON1, U2 HC-SR04

Commit message: Connector patch
Connections:
- net GND: now also P2.4 (P4); no longer P2.1 (P1)
- net P1: now also P2.2 (P2); no longer P2.3 (P3)
- net P2: now also P2.1 (P1); no longer P2.4 (P4)
- net VCC: now also P2.3 (P3); no longer P2.2 (P2)
Changed lines of the file:
@@
 LIBS:contrib
 LIBS:valves
+LIBS:MyLib-ALL
 LIBS:HC-SR04-cache
 EELAYER 25 0
@@
 encoding utf-8
 Sheet 1 1
-Title "Sensor HC-SR04 para Shield Sensor Base Grover GERSE"
+Title "Módulo Ultrasom HC-SR04 - Molex 2510 4 pinos "
 Date "2017-07-11"
 Rev "1.0"
-Comp "GERSE - Grupo de Estudos em Robótica e sistemas Embarcados"
-Comment1 "Facebook: www.facebook.com/gerserobot/ "
-Comment2 "Instagram: www.instagram.com/gerserobot/  "
-Comment3 "Website: gerserobotica.com"
-Comment4 "Projetista: @pedro_ibs (www.instagram.com/pedro_ibs/)"
+Comp "Shield Sensor Base Grover GERSE"
+Comment1 ""
+Comment2 ""
+Comment3 ""
+Comment4 ""
 $EndDescr
 $Comp
@@
 U 1 1 594A7B63
 P 4850 850
-F 0 "P2" H 4850 1100 50  0000 C CNN
+F 0 "P2" H 4850 600 50  0000 C CNN
 F 1 "CON1" V 4950 850 50  0000 C CNN
 F 2 "MY_kicad:molex_2510" H 4850 850 50  0001 C CNN
 F 3 "" H 4850 850 50  0000 C CNN
 	1    4850 850
-	0    -1   -1   0
+	0    1    -1   0
 $EndComp
 $Comp
