File: Conector molex 2510 4 pinos/LDR1/LDR_1.kicad_pcb (KiCad board)
At the start: 2 copper layers, 234 x 171 mm, 280 parts, among them P3 CON2

Commit message: Connector patch
Parts:
- removed the D1 at (139.8, 18.1)
- removed the D1 at (169.8, 168.1)
- removed the D1 at (169.8, 68.1)
- removed the D1 at (169.8, 93.1)
- removed the D1 at (169.8, 43.1)
- removed the D1 at (169.8, 18.1)
- removed the D1 at (229.8, 18.1)
- removed the D1 at (229.8, 43.1)
- removed the D1 at (229.8, 93.1)
- removed the D1 at (229.8, 68.1)
- removed the D1 at (229.8, 168.1)
- removed the D1 at (139.8, 43.1)
- removed the D1 at (229.8, 143.1)
- removed the D1 at (229.8, 118.1)
- removed the D1 at (199.8, 118.1)
- removed the D1 at (199.8, 143.1)
- removed the D1 at (199.8, 168.1)
- removed the D1 at (199.8, 68.1)
- removed the D1 at (199.8, 93.1)
- removed the D1 at (199.8, 43.1)
- removed the D1 at (199.8, 18.1)
- removed the D1 at (79.8, 18.1)
- removed the D1 at (139.8, 93.1)
- removed the D1 at (79.8, 43.1)
- removed the D1 at (79.8, 93.1)
- removed the D1 at (79.8, 68.1)
- removed the D1 at (79.8, 168.1)
- removed the D1 at (79.8, 143.1)
- removed the D1 at (79.8, 118.1)
- removed the D1 at (109.8, 118.1)
- removed the D1 at (109.8, 143.1)
- removed the D1 at (109.8, 168.1)
- removed the D1 at (109.8, 68.1)
- removed the D1 at (139.8, 68.1)
- removed the D1 at (109.8, 93.1)
- removed the D1 at (109.8, 43.1)
- removed the D1 at (109.8, 18.1)
- removed the D1 at (49.8, 18.1)
- removed the D1 at (49.8, 43.1)
- removed the D1 at (49.8, 93.1)
- removed the D1 at (49.8, 68.1)
- removed the D1 at (49.8, 168.1)
- removed the D1 at (49.8, 143.1)
- removed the D1 at (49.8, 118.1)
- removed the D1 at (139.8, 168.1)
- removed the D1 at (19.8, 118.1)
- removed the D1 at (19.8, 143.1)
- removed the D1 at (19.8, 168.1)
- removed the D1 at (19.8, 68.1)
- removed the D1 at (19.8, 93.1)
- removed the D1 at (19.8, 43.1)
- removed the D1 at (139.8, 143.1)
- removed the D1 at (139.8, 118.1)
- removed the D1 at (169.8, 118.1)
- removed the D1 at (169.8, 143.1)
- removed the P3 at (143.0, 32.6)
- removed the P3 at (173.0, 182.6)
- removed the P3 at (173.0, 82.6)
- removed the P3 at (173.0, 107.6)
- removed the P3 at (173.0, 57.6)
- removed the P3 at (173.0, 32.6)
- removed the P3 at (233.0, 32.6)
- removed the P3 at (233.0, 57.6)
- removed the P3 at (233.0, 107.6)
- removed the P3 at (233.0, 82.6)
- removed the P3 at (233.0, 182.6)
- removed the P3 at (143.0, 57.6)
- removed the P3 at (233.0, 157.6)
- removed the P3 at (233.0, 132.6)
- removed the P3 at (203.0, 132.6)
- removed the P3 at (203.0, 157.6)
- removed the P3 at (203.0, 182.6)
- removed the P3 at (203.0, 82.6)
- removed the P3 at (203.0, 107.6)
- removed the P3 at (203.0, 57.6)
- removed the P3 at (203.0, 32.6)
- removed the P3 at (83.0, 32.6)
- removed the P3 at (143.0, 107.6)
- removed the P3 at (83.0, 57.6)
- removed the P3 at (83.0, 107.6)
- removed the P3 at (83.0, 82.6)
- removed the P3 at (83.0, 182.6)
- removed the P3 at (83.0, 157.6)
- removed the P3 at (83.0, 132.6)
- removed the P3 at (113.0, 132.6)
- removed the P3 at (113.0, 157.6)
- removed the P3 at (113.0, 182.6)
- removed the P3 at (113.0, 82.6)
- removed the P3 at (143.0, 82.6)
- removed the P3 at (113.0, 107.6)
- removed the P3 at (113.0, 57.6)
- removed the P3 at (113.0, 32.6)
- removed the P3 at (53.0, 32.6)
- removed the P3 at (53.0, 57.6)
- removed the P3 at (53.0, 107.6)
- removed the P3 at (53.0, 82.6)
- removed the P3 at (53.0, 182.6)
- removed the P3 at (53.0, 157.6)
- removed the P3 at (53.0, 132.6)
- removed the P3 at (143.0, 182.6)
- removed the P3 at (23.0, 132.6)
- removed the P3 at (23.0, 157.6)
- removed the P3 at (23.0, 182.6)
- removed the P3 at (23.0, 82.6)
- removed the P3 at (23.0, 107.6)
- removed the P3 at (23.0, 57.6)
- removed the P3 at (143.0, 157.6)
- removed the P3 at (143.0, 132.6)
- removed the P3 at (173.0, 132.6)
- removed the P3 at (173.0, 157.6)
- removed the R2 at (143.6, 27.6)
- removed the R2 at (173.6, 177.6)
- removed the R2 at (173.6, 77.6)
- removed the R2 at (173.6, 102.6)
- removed the R2 at (173.6, 52.6)
- removed the R2 at (173.6, 27.6)
- removed the R2 at (233.6, 27.6)
- removed the R2 at (233.6, 52.6)
- removed the R2 at (233.6, 102.6)
- removed the R2 at (233.6, 77.6)
- removed the R2 at (233.6, 177.6)
- removed the R2 at (143.6, 52.6)
- removed the R2 at (233.6, 152.6)
- removed the R2 at (233.6, 127.6)
- removed the R2 at (203.6, 127.6)
- removed the R2 at (203.6, 152.6)
- removed the R2 at (203.6, 177.6)
- removed the R2 at (203.6, 77.6)
- removed the R2 at (203.6, 102.6)
- removed the R2 at (203.6, 52.6)
- removed the R2 at (203.6, 27.6)
- removed the R2 at (83.6, 27.6)
- removed the R2 at (143.6, 102.6)
- removed the R2 at (83.6, 52.6)
- removed the R2 at (83.6, 102.6)
- removed the R2 at (83.6, 77.6)
- removed the R2 at (83.6, 177.6)
- removed the R2 at (83.6, 152.6)
- removed the R2 at (83.6, 127.6)
- removed the R2 at (113.6, 127.6)
- removed the R2 at (113.6, 152.6)
- removed the R2 at (113.6, 177.6)
- removed the R2 at (113.6, 77.6)
- removed the R2 at (143.6, 77.6)
- removed the R2 at (113.6, 102.6)
- removed the R2 at (113.6, 52.6)
- removed the R2 at (113.6, 27.6)
- removed the R2 at (53.6, 27.6)
- removed the R2 at (53.6, 52.6)
- removed the R2 at (53.6, 102.6)
- removed the R2 at (53.6, 77.6)
- removed the R2 at (53.6, 177.6)
- removed the R2 at (53.6, 152.6)
- removed the R2 at (53.6, 127.6)
- removed the R2 at (143.6, 177.6)
- removed the R2 at (23.6, 127.6)
- removed the R2 at (23.6, 152.6)
- removed the R2 at (23.6, 177.6)
- removed the R2 at (23.6, 77.6)
- removed the R2 at (23.6, 102.6)
- removed the R2 at (23.6, 52.6)
- removed the R2 at (143.6, 152.6)
- removed the R2 at (143.6, 127.6)
- removed the R2 at (173.6, 127.6)
- removed the R2 at (173.6, 152.6)
- removed the R3 at (143.6, 18.1)
- removed the R3 at (173.6, 168.1)
- removed the R3 at (173.6, 68.1)
- removed the R3 at (173.6, 93.1)
- removed the R3 at (173.6, 43.1)
- removed the R3 at (173.6, 18.1)
- removed the R3 at (233.6, 18.1)
- removed the R3 at (233.6, 43.1)
- removed the R3 at (233.6, 93.1)
- removed the R3 at (233.6, 68.1)
- removed the R3 at (233.6, 168.1)
- removed the R3 at (143.6, 43.1)
- removed the R3 at (233.6, 143.1)
- removed the R3 at (233.6, 118.1)
- removed the R3 at (203.6, 118.1)
- removed the R3 at (203.6, 143.1)
- removed the R3 at (203.6, 168.1)
- removed the R3 at (203.6, 68.1)
- removed the R3 at (203.6, 93.1)
- removed the R3 at (203.6, 43.1)
- removed the R3 at (203.6, 18.1)
- removed the R3 at (83.6, 18.1)
- removed the R3 at (143.6, 93.1)
- removed the R3 at (83.6, 43.1)
- removed the R3 at (83.6, 93.1)
- removed the R3 at (83.6, 68.1)
- removed the R3 at (83.6, 168.1)
- removed the R3 at (83.6, 143.1)
- removed the R3 at (83.6, 118.1)
- removed the R3 at (113.6, 118.1)
- removed the R3 at (113.6, 143.1)
- removed the R3 at (113.6, 168.1)
- removed the R3 at (113.6, 68.1)
- removed the R3 at (143.6, 68.1)
- removed the R3 at (113.6, 93.1)
- removed the R3 at (113.6, 43.1)
- removed the R3 at (113.6, 18.1)
- removed the R3 at (53.6, 18.1)
- removed the R3 at (53.6, 43.1)
- removed the R3 at (53.6, 93.1)
- removed the R3 at (53.6, 68.1)
- removed the R3 at (53.6, 168.1)
- removed the R3 at (53.6, 143.1)
- removed the R3 at (53.6, 118.1)
- removed the R3 at (143.6, 168.1)
- removed the R3 at (23.6, 118.1)
- removed the R3 at (23.6, 143.1)
- removed the R3 at (23.6, 168.1)
- removed the R3 at (23.6, 68.1)
- removed the R3 at (23.6, 93.1)
- removed the R3 at (23.6, 43.1)
- removed the R3 at (143.6, 143.1)
- removed the R3 at (143.6, 118.1)
- removed the R3 at (173.6, 118.1)
- removed the R3 at (173.6, 143.1)
- removed the R4 at (150.6, 23.2)
- removed the R4 at (180.6, 173.2)
- removed the R4 at (180.6, 73.2)
- removed the R4 at (180.6, 98.2)
- removed the R4 at (180.6, 48.2)
- removed the R4 at (180.6, 23.2)
- removed the R4 at (240.6, 23.2)
- removed the R4 at (240.6, 48.2)
- removed the R4 at (240.6, 98.2)
- removed the R4 at (240.6, 73.2)
- removed the R4 at (240.6, 173.2)
- removed the R4 at (150.6, 48.2)
- removed the R4 at (240.6, 148.2)
- removed the R4 at (240.6, 123.2)
- removed the R4 at (210.6, 123.2)
- removed the R4 at (210.6, 148.2)
- removed the R4 at (210.6, 173.2)
- removed the R4 at (210.6, 73.2)
- removed the R4 at (210.6, 98.2)
- removed the R4 at (210.6, 48.2)
- removed the R4 at (210.6, 23.2)
- removed the R4 at (90.6, 23.2)
- removed the R4 at (150.6, 98.2)
- removed the R4 at (90.6, 48.2)
- removed the R4 at (90.6, 98.2)
- removed the R4 at (90.6, 73.2)
- removed the R4 at (90.6, 173.2)
- removed the R4 at (90.6, 148.2)
- removed the R4 at (90.6, 123.2)
- removed the R4 at (120.6, 123.2)
- removed the R4 at (120.6, 148.2)
- removed the R4 at (120.6, 173.2)
- removed the R4 at (120.6, 73.2)
- removed the R4 at (150.6, 73.2)
- removed the R4 at (120.6, 98.2)
- removed the R4 at (120.6, 48.2)
- removed the R4 at (120.6, 23.2)
- removed the R4 at (60.6, 23.2)
- removed the R4 at (60.6, 48.2)
- removed the R4 at (60.6, 98.2)
- removed the R4 at (60.6, 73.2)
- removed the R4 at (60.6, 173.2)
- removed the R4 at (60.6, 148.2)
- removed the R4 at (60.6, 123.2)
- removed the R4 at (150.6, 173.2)
- removed the R4 at (30.6, 123.2)
- removed the R4 at (30.6, 148.2)
- removed the R4 at (30.6, 173.2)
- removed the R4 at (30.6, 73.2)
- removed the R4 at (30.6, 98.2)
- removed the R4 at (30.6, 48.2)
- removed the R4 at (150.6, 148.2)
- removed the R4 at (150.6, 123.2)
- removed the R4 at (180.6, 123.2)
- removed the R4 at (180.6, 148.2)
- moved P3 0.20 mm to (23.0, 32.4)
Routing:
- net P4: track 713.7 -> 12.7 mm
- net P3: track 707.5 -> 12.6 mm
- net VCC: track 556.8 -> 9.94 mm
- net Net-(D1-Pad1): track 213.4 -> 3.81 mm
Other:
- board size 234 x 171 mm -> 24 x 21 mm
- board text removed: "Necessário espelhar Need to mirror"
