File: Conector molex 2510 4 pinos/Potenciômetro/POT.kicad_pcb (KiCad board)
At the start: 2 copper layers, 235 x 140 mm, 64 parts, among them P5 CON4

Commit message: Connector patch
Parts:
- removed the P5 at (143.4, 45.8)
- removed the P5 at (233.4, 85.8)
- removed the P5 at (233.4, 125.8)
- removed the P5 at (233.4, 165.8)
- removed the P5 at (203.4, 165.8)
- removed the P5 at (203.4, 125.8)
- removed the P5 at (203.4, 85.8)
- removed the P5 at (203.4, 45.8)
- removed the P5 at (83.4, 45.8)
- removed the P5 at (83.4, 85.8)
- removed the P5 at (83.4, 125.8)
- removed the P5 at (143.4, 85.8)
- removed the P5 at (83.4, 165.8)
- removed the P5 at (113.4, 165.8)
- removed the P5 at (113.4, 125.8)
- removed the P5 at (113.4, 85.8)
- removed the P5 at (113.4, 45.8)
- removed the P5 at (53.4, 45.8)
- removed the P5 at (53.4, 85.8)
- removed the P5 at (53.4, 125.8)
- removed the P5 at (53.4, 165.8)
- removed the P5 at (23.4, 165.8)
- removed the P5 at (143.4, 125.8)
- removed the P5 at (23.4, 125.8)
- removed the P5 at (23.4, 85.8)
- removed the P5 at (143.4, 165.8)
- removed the P5 at (173.4, 165.8)
- removed the P5 at (173.4, 125.8)
- removed the P5 at (173.4, 85.8)
- removed the P5 at (173.4, 45.8)
- removed the P5 at (233.4, 45.8)
- removed the RV2 at (143.0, 35.0)
- removed the RV2 at (233.0, 75.0)
- removed the RV2 at (233.0, 115.0)
- removed the RV2 at (233.0, 155.0)
- removed the RV2 at (203.0, 155.0)
- removed the RV2 at (203.0, 115.0)
- removed the RV2 at (203.0, 75.0)
- removed the RV2 at (203.0, 35.0)
- removed the RV2 at (83.0, 35.0)
- removed the RV2 at (83.0, 75.0)
- removed the RV2 at (83.0, 115.0)
- removed the RV2 at (143.0, 75.0)
- removed the RV2 at (83.0, 155.0)
- removed the RV2 at (113.0, 155.0)
- removed the RV2 at (113.0, 115.0)
- removed the RV2 at (113.0, 75.0)
- removed the RV2 at (113.0, 35.0)
- removed the RV2 at (53.0, 35.0)
- removed the RV2 at (53.0, 75.0)
- removed the RV2 at (53.0, 115.0)
- removed the RV2 at (53.0, 155.0)
- removed the RV2 at (23.0, 155.0)
- removed the RV2 at (143.0, 115.0)
- removed the RV2 at (23.0, 115.0)
- removed the RV2 at (23.0, 75.0)
- removed the RV2 at (143.0, 155.0)
- removed the RV2 at (173.0, 155.0)
- removed the RV2 at (173.0, 115.0)
- removed the RV2 at (173.0, 75.0)
- removed the RV2 at (173.0, 35.0)
- removed the RV2 at (233.0, 35.0)
Routing:
- net P7: track 931.5 -> 29.1 mm
- net VCC: track 424.4 -> 13.3 mm
Other:
- board size 235 x 140 mm -> 25 x 20 mm
- board text removed: "Necessário espelhar Need to mirror"
